File: ESPP.sch (KiCad schematic (older format))
At the start: 18 parts, among them P1 USB_OTG, Q1 MMBT3904, Q2 MMBT3904, U1 RT9193, U2 CH340G, X1 12MHz, X2 ESP-PROG

Commit message: WIP
Parts:
- added D1: BAT54C, TO_SOT_Packages_SMD:SOT-23, symbol D_Schottky_x2_KCom_AAK
- C3: value 47u -> 1u
Connections:
- net labels removed: 5V
- wire segments 33 -> 35
- no-connect marks 6 -> 7
Changed lines of the file:
@@
 LIBS:valves
 LIBS:device.farm
+LIBS:ESPP-cache
 EELAYER 25 0
 EELAYER END
@@
 P 4300 5050
 F 0 "C3" H 4415 5096 50  0000 L CNN
-F 1 "47u" H 4415 5005 50  0000 L CNN
+F 1 "1u" H 4415 5005 50  0000 L CNN
 F 2 "Capacitors_SMD:C_0805" H 4338 4900 50  0001 C CNN
 F 3 "" H 4300 5050 50  0000 C CNN
@@
 	1    0    0    -1
 $EndComp
-Text Label 2750 4800 0    60   ~ 0
-5V
 $Comp
 L CH340G U2
@@
 	1    0    0    -1
 $EndComp
-$Comp
-L VCC #PWR018
-U 1 1 5A9A0ECA
-P 8600 1800
-F 0 "#PWR018" H 8600 1650 50  0001 C CNN
-F 1 "VCC" V 8618 1927 50  0000 L CNN
-F 2 "" H 8600 1800 50  0000 C CNN
-F 3 "" H 8600 1800 50  0000 C CNN
-	1    8600 1800
-	0    -1   -1   0
-$EndComp
 Text Label 8600 1950 2    60   ~ 0
 RESET
@@
 TX
 $Comp
-L VCC #PWR019
+L VCC #PWR018
 U 1 1 5A9A158D
 P 2900 1950
-F 0 "#PWR019" H 2900 1800 50  0001 C CNN
+F 0 "#PWR018" H 2900 1800 50  0001 C CNN
 F 1 "VCC" V 2900 2150 50  0000 C CNN
 F 2 "" H 2900 1950 50  0001 C CNN
@@
 $EndComp
 $Comp
-L PWR_FLAG #FLG020
+L PWR_FLAG #FLG019
 U 1 1 5A9A15D5
 P 2900 1950
-F 0 "#FLG020" H 2900 2025 50  0001 C CNN
+F 0 "#FLG019" H 2900 2025 50  0001 C CNN
 F 1 "PWR_FLAG" V 2900 2250 50  0000 C CNN
 F 2 "" H 2900 1950 50  0001 C CNN
@@
 	0    -1   -1   0
 $EndComp
+$Comp
+L D_Schottky_x2_KCom_AAK D1
+U 1 1 5A9B6F57
+P 8500 1400
+F 0 "D1" H 8550 1300 50  0000 C CNN
+F 1 "BAT54C" H 8500 1500 50  0000 C CNN
+F 2 "TO_SOT_Packages_SMD:SOT-23" H 8500 1400 50  0001 C CNN
+F 3 "" H 8500 1400 50  0001 C CNN
+	1    8500 1400
+	1    0    0    -1
+$EndComp
+Wire Wire Line
+	8500 1600 8500 1800
+Wire Wire Line
+	8500 1800 8600 1800
+NoConn ~ 8800 1400
+$Comp
+L VCC #PWR020
+U 1 1 5A9A0ECA
+P 8200 1400
+F 0 "#PWR020" H 8200 1250 50  0001 C CNN
+F 1 "VCC" V 8218 1527 50  0000 L CNN
+F 2 "" H 8200 1400 50  0000 C CNN
+F 3 "" H 8200 1400 50  0000 C CNN
+	1    8200 1400
+	0    -1   -1   0
+$EndComp
