File: ESPP.sch (KiCad schematic (older format))
At the start: 19 parts, among them P1 USB_OTG, Q1 MMBT3904, Q2 MMBT3904, U1 RT9193, U2 CH340G, X1 12MHz, X2 ESP-PROG

Commit message: WIP
Parts:
- removed U2: CH340G, SMD_Packages:SO-16-N, symbol CH340G
- added U2: CH340G, Package_SO:SOIC-16_3.9x9.9mm_P1.27mm, symbol Interface_USB:CH340G
- C1, C2, C3, C4, C5, C6: footprint Capacitors_SMD:C_0805 -> Capacitor_SMD:C_0805_2012Metric; symbol C -> Device:C
- D1: footprint TO_SOT_Packages_SMD:SOT-23 -> Package_TO_SOT_SMD:SOT-23; symbol D_Schottky_x2_KCom_AAK -> Device:D_Schottky_x2_KCom_AAK
- L1: footprint Resistors_SMD:R_0805 -> Inductor_SMD:L_0805_2012Metric; symbol Ferrite_Bead -> Device:Ferrite_Bead
- P1: symbol USB_OTG -> Connector:USB_OTG
- Q1, Q2: footprint TO_SOT_Packages_SMD:SOT-23 -> Package_TO_SOT_SMD:SOT-23; symbol MMBT3904 -> Transistor_BJT:MMBT3904
- R1, R2, R3, R4: footprint Resistors_SMD:R_0805 -> Resistor_SMD:R_0805_2012Metric; symbol R -> Device:R
- U1: footprint TO_SOT_Packages_SMD:SOT-23-5 -> Package_TO_SOT_SMD:SOT-23-5; symbol RT9193 -> device.farm:RT9193
- X1: footprint Crystals:Crystal_SMD_SeikoEpson_TSX3225-4pin_3.2x2.5mm -> Crystal:Crystal_SMD_3225-4Pin_3.2x2.5mm; symbol Crystal_GND24 -> Device:Crystal_GND24
- X2: symbol ESP-PROG -> device.farm:ESP-PROG
Connections:
- wire segments 35 -> 44
