File: ESPP.kicad_pcb (KiCad board)
At the start: 2 copper layers, 32 x 18 mm, 20 parts, among them P1 USB_OTG, Q1 MMBT3904, Q2 MMBT3904, U1 RT9193, U2 CH340G, X1 12MHz, X2 ESP-PROG

Commit message: WIP
Parts:
- P1: footprint device.farm:conn_usb_B_micro_smd-2 -> Drake:conn_usb_B_micro_smd-2
- X2: footprint device.farm:Micro-Match-FOB-6 -> Drake:Micro-Match-FOB-6
